File: toro-pcb/toro-pcb.kicad_sch (KiCad schematic)
At the start: 140 parts, among them SW1 Kailh_socket, SW10 Kailh_socket, SW11 Kailh_socket, SW12 Kailh_socket, SW13 Kailh_socket, SW14 Kailh_socket, SW15 Kailh_socket, SW16 Kailh_socket, SW17 Kailh_socket, SW18 Kailh_socket, SW19 Kailh_socket, SW2 RotaryEncoder_Switch, SW20 Kailh_socket, SW21 Kailh_socket, SW22 Kailh_socket, SW23 Kailh_socket, SW24 Kailh_socket, SW25 Kailh_socket, SW26 Kailh_socket, SW27 Kailh_socket, SW28 Kailh_socket, SW29 Kailh_socket, SW3 Kailh_socket, SW30 Kailh_socket, SW31 Kailh_socket, SW32 Kailh_socket, SW33 Kailh_socket, SW34 Kailh_socket, SW35 Kailh_socket, SW36 Kailh_socket, SW37 Kailh_socket, SW38 Kailh_socket, SW4 Kailh_socket, SW40 Kailh_socket, SW41 Kailh_socket, SW42 Kailh_socket, SW43 Kailh_socket, SW44 Kailh_socket, SW45 Kailh_socket, SW46 Kailh_socket, SW47 Kailh_socket, SW48 Kailh_socket, SW49 Kailh_socket, SW5 Kailh_socket, SW51 Kailh_socket, SW52 Kailh_socket, SW53 Kailh_socket, SW54 Kailh_socket, SW55 Kailh_socket, SW56 Kailh_socket, SW57 Kailh_socket, SW58 Kailh_socket, SW59 Kailh_socket, SW6 Kailh_socket, SW60 Kailh_socket, SW61 Kailh_socket, SW62 Kailh_socket, SW63 Kailh_socket, SW64 Kailh_socket, SW65 Kailh_socket, SW67 Kailh_socket, SW68 Kailh_socket, SW69 Kailh_socket, SW7 Kailh_socket, SW71 Kailh_socket, SW72 Kailh_socket, SW73 Kailh_socket, SW8 Kailh_socket, SW9 Kailh_socket, U2 SC0917

Commit message: #ididntsavemychanges. rotary encoder
Parts:
- removed D66: 1N4148, Diode_THT:D_DO-35_SOD27_P7.62mm_Horizontal, symbol Diode:1N4148
Connections:
- net Col 0: now also U2.7 (GP5)
- net Col 1: now also U2.9 (GP6)
- net Col 10: now also U2.20 (GP15)
- net Col 11: now also U2.21 (GP16)
- net Col 12: now also U2.22 (GP17)
- net Col 13: now also U2.24 (GP18)
- net Col 14: now also U2.25 (GP19)
- net Col 15: now also U2.26 (GP20)
- net Col 16: now also U2.27 (GP21)
- net Col 17: now also U2.29 (GP22); no longer SW2.A, SW2.B, SW2.C
- net Col 2: now also U2.10 (GP7)
- net Col 3: now also U2.11 (GP8)
- net Col 4: now also U2.12 (GP9)
- net Col 5: now also U2.14 (GP10)
- net Col 6: now also U2.15 (GP11)
- net Col 7: now also U2.16 (GP12)
- net Col 8: now also U2.17 (GP13)
- net Col 9: now also U2.19 (GP14)
- net Row 0: now also U2.1 (GP0)
- net Row 1: now also U2.2 (GP1)
- net Row 2: now also U2.4 (GP2)
- net Row 3: now also U2.5 (GP3)
- net Row 4: now also U2.6 (GP4)
- net ENC_A: now reaches U2.31 (GP26)
- net ENC_A: now also SW2.A
- net ENC_B: now reaches U2.32 (GP27)
- net ENC_B: now also SW2.B
- net ENC_S1: now reaches U2.34 (GP28)
- net ENC_S1: now also SW2.S1
- net GND: now reaches SW2.S2
- net GND: now also SW2.C
Other:
- note added: "Rotary encoder"
- note added: "Switch Matrix"
- moved on the sheet: D1

Commit message: led strip
Parts:
- removed D1: SK6812MINI, LED_SMD:LED_SK6812MINI_PLCC4_3.5x3.5mm_P1.75mm, symbol LED:SK6812MINI
- removed U2: SC0917, SC0917:MODULE_SC0917, symbol SC0917:SC0917
- added D1, D137, D138, D139, D140, D141, D142, D143, D144, D145, D146, D147, D148, D149, D150, D151, D152, D153, D154, D155, D156, D157, D158, D159, D160, D161, D162, D163, D164, D165, D166, D167, D168, D169, D170, D171, D172, D173, D174, D175, D176, D177, D178, D179, D180, D181, D182, D183, D184, D185, D186, D187, D188, D189, D190, D191, D192, D193, D194, D195, D196, D197, D39, D50, D66, D67, D71, D75: NeoPixel_THT, symbol LED:NeoPixel_THT
- added U1: Pico, RPi_Pico:RPi_Pico_SMD_TH, symbol MCU_RaspberryPi_and_Boards:Pico
Connections:
- net Col 17 is gone; now on net Col 16: SW61.1, SW63.1, SW64.1, SW65.1
- net Col 0: now also SW15.1, SW21.1, SW27.1, SW9.1, U1.7 (GPIO5)
- net Col 1: now also SW10.1, SW16.1, SW22.1, U1.9 (GPIO6); no longer SW15.1, SW21.1, SW27.1, SW9.1
- net Col 10: now also SW46.1, SW49.1, SW55.1, U1.19 (GPIO14); no longer SW44.1, SW47.1, SW54.1
- net Col 11: now also SW48.1, SW68.1, SW69.1, U1.21 (GPIO16); no longer SW46.1, SW49.1, SW55.1
- net Col 12: now also SW67.1, SW72.1, SW73.1, U1.22 (GPIO17); no longer SW48.1, SW68.1, SW69.1
- net Col 13: now also SW71.1, U1.24 (GPIO18); no longer SW67.1, SW72.1, SW73.1
- net Col 14: now also SW59.1, U1.25 (GPIO19); no longer SW71.1
- net Col 15: now also SW60.1, SW62.1, U1.26 (GPIO20); no longer SW59.1
- net Col 16: now also U1.27 (GPIO21); no longer SW60.1, SW62.1
- net Col 2: now also SW11.1, SW17.1, SW23.1, U1.10 (GPIO7); no longer SW10.1, SW16.1, SW22.1
- net Col 3: now also SW12.1, SW18.1, SW24.1, SW30.1, U1.11 (GPIO8); no longer SW11.1, SW17.1, SW23.1
- net Col 4: now also SW13.1, SW19.1, SW25.1, SW31.1, U1.12 (GPIO9); no longer SW12.1, SW18.1, SW24.1, SW30.1
- net Col 5: now also SW14.1, SW20.1, SW26.1, SW32.1, U1.14 (GPIO10); no longer SW13.1, SW19.1, SW25.1, SW31.1
- net Col 6: now also SW38.1, SW41.1, SW51.1, SW56.1, U1.15 (GPIO11); no longer SW14.1, SW20.1, SW26.1, SW32.1
- net Col 7: now also SW40.1, SW43.1, SW52.1, SW57.1, U1.16 (GPIO12); no longer SW38.1, SW41.1, SW51.1, SW56.1
- net Col 8: now also SW42.1, SW45.1, SW53.1, SW58.1, U1.17 (GPIO13); no longer SW40.1, SW43.1, SW52.1, SW57.1
- net Col 9: now also SW44.1, SW47.1, SW54.1, U1.20 (GPIO15); no longer SW42.1, SW45.1, SW53.1, SW58.1
- net ENC_A: now also U1.29 (GPIO22)
- net ENC_B: now also U1.31 (GPIO26_ADC0)
- net ENC_S1: now also U1.32 (GPIO27_ADC1)
- net GND: now also D1.2 (GND), D137.2 (GND), D138.2 (GND), D139.2 (GND), D140.2 (GND), D141.2 (GND), D142.2 (GND), D143.2 (GND), D144.2 (GND), D145.2 (GND), D146.2 (GND), D147.2 (GND), D148.2 (GND), D149.2 (GND), D150.2 (GND), D151.2 (GND), D152.2 (GND), D153.2 (GND), D154.2 (GND), D155.2 (GND), D156.2 (GND), D157.2 (GND), D158.2 (GND), D159.2 (GND), D160.2 (GND), D161.2 (GND), D162.2 (GND), D163.2 (GND), D164.2 (GND), D165.2 (GND), D166.2 (GND), D167.2 (GND), D168.2 (GND), D169.2 (GND), D170.2 (GND), D171.2 (GND), D172.2 (GND), D173.2 (GND), D174.2 (GND), D175.2 (GND), D176.2 (GND), D177.2 (GND), D178.2 (GND), D179.2 (GND), D180.2 (GND), D181.2 (GND), D182.2 (GND), D183.2 (GND), D184.2 (GND), D185.2 (GND), D186.2 (GND), D187.2 (GND), D188.2 (GND), D189.2 (GND), D190.2 (GND), D191.2 (GND), D192.2 (GND), D193.2 (GND), D194.2 (GND), D195.2 (GND), D196.2 (GND), D197.2 (GND), D39.2 (GND), D50.2 (GND), D66.2 (GND), D67.2 (GND), D71.2 (GND), D75.2 (GND)
- net Row 0: now also U1.1 (GPIO0)
- net Row 1: now also U1.2 (GPIO1)
- net Row 2: now also U1.4 (GPIO2)
- net Row 3: now also U1.5 (GPIO3)
- net Row 4: now also U1.6 (GPIO4)
- new net: D1.1 (DOUT), D1.4 (DIN), D137.1 (DOUT), D137.4 (DIN), D138.1 (DOUT), D138.4 (DIN), D142.1 (DOUT), D142.4 (DIN), D145.1 (DOUT), D145.4 (DIN), D146.1 (DOUT), D146.4 (DIN), D150.1 (DOUT), D150.4 (DIN), D151.1 (DOUT), D151.4 (DIN), D155.1 (DOUT), D155.4 (DIN), D156.1 (DOUT), D156.4 (DIN), D160.1 (DOUT), D160.4 (DIN), D161.1 (DOUT), D161.4 (DIN), D164.1 (DOUT), D164.4 (DIN), D165.1 (DOUT), D165.4 (DIN), D166.1 (DOUT), D166.4 (DIN), D169.1 (DOUT), D169.4 (DIN), D170.1 (DOUT), D170.4 (DIN), D173.1 (DOUT), D173.4 (DIN), D174.1 (DOUT), D174.4 (DIN), D178.1 (DOUT), D178.4 (DIN), D179.1 (DOUT), D179.4 (DIN), D183.1 (DOUT), D183.4 (DIN), D184.1 (DOUT), D184.4 (DIN), D188.1 (DOUT), D188.4 (DIN), D196.1 (DOUT), D39.1 (DOUT), D39.4 (DIN), D67.1 (DOUT), D67.4 (DIN), D71.1 (DOUT), D71.4 (DIN), D75.1 (DOUT), D75.4 (DIN)
- new net: D139.1 (DOUT), D143.1 (DOUT), D143.4 (DIN), D147.1 (DOUT), D147.4 (DIN), D152.1 (DOUT), D152.4 (DIN), D157.1 (DOUT), D157.4 (DIN), D162.1 (DOUT), D162.4 (DIN), D167.1 (DOUT), D167.4 (DIN), D171.1 (DOUT), D171.4 (DIN), D175.1 (DOUT), D175.4 (DIN), D180.1 (DOUT), D180.4 (DIN), D185.1 (DOUT), D185.4 (DIN), D189.1 (DOUT), D189.4 (DIN), D196.4 (DIN), D197.1 (DOUT), D197.4 (DIN), D50.1 (DOUT), D50.4 (DIN)
- new net +5V: D1.3 (VDD), D137.3 (VDD), D138.3 (VDD), D139.3 (VDD), D140.3 (VDD), D141.3 (VDD), D142.3 (VDD), D143.3 (VDD), D144.3 (VDD), D145.3 (VDD), D146.3 (VDD), D147.3 (VDD), D148.3 (VDD), D149.3 (VDD), D150.3 (VDD), D151.3 (VDD), D152.3 (VDD), D153.3 (VDD), D154.3 (VDD), D155.3 (VDD), D156.3 (VDD), D157.3 (VDD), D158.3 (VDD), D159.3 (VDD), D160.3 (VDD), D161.3 (VDD), D162.3 (VDD), D163.3 (VDD), D164.3 (VDD), D165.3 (VDD), D166.3 (VDD), D167.3 (VDD), D168.3 (VDD), D169.3 (VDD), D170.3 (VDD), D171.3 (VDD), D172.3 (VDD), D173.3 (VDD), D174.3 (VDD), D175.3 (VDD), D176.3 (VDD), D177.3 (VDD), D178.3 (VDD), D179.3 (VDD), D180.3 (VDD), D181.3 (VDD), D182.3 (VDD), D183.3 (VDD), D184.3 (VDD), D185.3 (VDD), D186.3 (VDD), D187.3 (VDD), D188.3 (VDD), D189.3 (VDD), D190.3 (VDD), D191.3 (VDD), D192.3 (VDD), D193.3 (VDD), D194.3 (VDD), D195.3 (VDD), D196.3 (VDD), D197.3 (VDD), D39.3 (VDD), D50.3 (VDD), D66.3 (VDD), D67.3 (VDD), D71.3 (VDD), D75.3 (VDD)
- new net LEDS: D139.4 (DIN), D140.1 (DOUT), D140.4 (DIN), D141.1 (DOUT), D141.4 (DIN), D144.1 (DOUT), D144.4 (DIN), D148.1 (DOUT), D148.4 (DIN), D149.1 (DOUT), D149.4 (DIN), D153.1 (DOUT), D153.4 (DIN), D154.1 (DOUT), D154.4 (DIN), D158.1 (DOUT), D158.4 (DIN), D159.1 (DOUT), D159.4 (DIN), D163.1 (DOUT), D163.4 (DIN), D168.1 (DOUT), D168.4 (DIN), D172.1 (DOUT), D172.4 (DIN), D176.1 (DOUT), D176.4 (DIN), D177.1 (DOUT), D177.4 (DIN), D181.1 (DOUT), D181.4 (DIN), D182.1 (DOUT), D182.4 (DIN), D186.1 (DOUT), D186.4 (DIN), D187.1 (DOUT), D187.4 (DIN), D190.1 (DOUT), D190.4 (DIN), D191.1 (DOUT), D191.4 (DIN), D192.1 (DOUT), D192.4 (DIN), D193.1 (DOUT), D193.4 (DIN), D194.1 (DOUT), D194.4 (DIN), D195.1 (DOUT), D195.4 (DIN), D66.1 (DOUT), D66.4 (DIN), U1.34 (GPIO28_ADC2)
Other:
- note added: "Led String"
- note added: "Rotary Encoder"
- note removed: "Rotary encoder"
- moved on the sheet: D10, D11, D12, D13, D14, D15, D16, D17, D18, D19, D2, D20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

Commit message: peeceebee
Parts:
- removed D137, D138, D139, D140, D141, D142, D143, D144, D145, D146, D147, D148, D149, D150, D151, D152, D153, D154, D155, D156, D157, D158, D159, D160, D161, D162, D163, D164, D165, D166, D167, D168, D169, D170, D171, D172, D173, D174, D175, D176, D177, D178, D179, D180, D181, D182, D183, D184, D185, D186, D187, D188, D189, D190, D191, D192, D193, D194, D195, D196, D197, D71, D75: NeoPixel_THT, symbol LED:NeoPixel_THT
- added D100, D101, D102, D103, D104, D105, D106, D107, D108, D109, D110, D111, D112, D113, D114, D115, D116, D117, D118, D119, D120, D121, D122, D123, D124, D125, D126, D127, D128, D129, D130, D131, D132, D133, D134, D135, D136, D198, D199, D76, D77, D78, D79, D80, D81, D82, D83, D84, D85, D86, D87, D88, D89, D90, D91, D92, D93, D94, D95, D96, D97, D98, D99: NeoPixel_THT, LED_SMD:LED_SK6812MINI_PLCC4_3.5x3.5mm_P1.75mm, symbol LED:NeoPixel_THT
- D1, D39, D50, D66, D67: footprint (none) -> LED_SMD:LED_SK6812MINI_PLCC4_3.5x3.5mm_P1.75mm
Connections:
- net +5V: now also D100.3 (VDD), D101.3 (VDD), D102.3 (VDD), D103.3 (VDD), D104.3 (VDD), D105.3 (VDD), D106.3 (VDD), D107.3 (VDD), D108.3 (VDD), D109.3 (VDD), D110.3 (VDD), D111.3 (VDD), D112.3 (VDD), D113.3 (VDD), D114.3 (VDD), D115.3 (VDD), D116.3 (VDD), D117.3 (VDD), D118.3 (VDD), D119.3 (VDD), D120.3 (VDD), D121.3 (VDD), D122.3 (VDD), D123.3 (VDD), D124.3 (VDD), D125.3 (VDD), D126.3 (VDD), D127.3 (VDD), D128.3 (VDD), D129.3 (VDD), D130.3 (VDD), D131.3 (VDD), D132.3 (VDD), D133.3 (VDD), D134.3 (VDD), D135.3 (VDD), D136.3 (VDD), D198.3 (VDD), D199.3 (VDD), D76.3 (VDD), D77.3 (VDD), D78.3 (VDD), D79.3 (VDD), D80.3 (VDD), D81.3 (VDD), D82.3 (VDD), D83.3 (VDD), D84.3 (VDD), D85.3 (VDD), D86.3 (VDD), D87.3 (VDD), D88.3 (VDD), D89.3 (VDD), D90.3 (VDD), D91.3 (VDD), D92.3 (VDD), D93.3 (VDD), D94.3 (VDD), D95.3 (VDD), D96.3 (VDD), D97.3 (VDD), D98.3 (VDD), D99.3 (VDD)
- net GND: now also D100.2 (GND), D101.2 (GND), D102.2 (GND), D103.2 (GND), D104.2 (GND), D105.2 (GND), D106.2 (GND), D107.2 (GND), D108.2 (GND), D109.2 (GND), D110.2 (GND), D111.2 (GND), D112.2 (GND), D113.2 (GND), D114.2 (GND), D115.2 (GND), D116.2 (GND), D117.2 (GND), D118.2 (GND), D119.2 (GND), D120.2 (GND), D121.2 (GND), D122.2 (GND), D123.2 (GND), D124.2 (GND), D125.2 (GND), D126.2 (GND), D127.2 (GND), D128.2 (GND), D129.2 (GND), D130.2 (GND), D131.2 (GND), D132.2 (GND), D133.2 (GND), D134.2 (GND), D135.2 (GND), D136.2 (GND), D198.2 (GND), D199.2 (GND), D76.2 (GND), D77.2 (GND), D78.2 (GND), D79.2 (GND), D80.2 (GND), D81.2 (GND), D82.2 (GND), D83.2 (GND), D84.2 (GND), D85.2 (GND), D86.2 (GND), D87.2 (GND), D88.2 (GND), D89.2 (GND), D90.2 (GND), D91.2 (GND), D92.2 (GND), D93.2 (GND), D94.2 (GND), D95.2 (GND), D96.2 (GND), D97.2 (GND), D98.2 (GND), D99.2 (GND)
- net LEDS: now also D67.1 (DOUT), D67.4 (DIN), D103.1 (DOUT), D103.4 (DIN), D108.1 (DOUT), D108.4 (DIN), D113.1 (DOUT), D113.4 (DIN), D132.1 (DOUT), D132.4 (DIN), D133.1 (DOUT), D133.4 (DIN), D134.1 (DOUT), D134.4 (DIN), D136.1 (DOUT), D80.1 (DOUT), D80.4 (DIN), D93.1 (DOUT), D93.4 (DIN), D98.1 (DOUT), D98.4 (DIN); no longer D66.1 (DOUT), D66.4 (DIN)
- net at D50.1 (DOUT), D50.4 (DIN): now also D39.1 (DOUT), D39.4 (DIN), D66.1 (DOUT), D66.4 (DIN), D100.1 (DOUT), D100.4 (DIN), D101.1 (DOUT), D101.4 (DIN), D102.1 (DOUT), D102.4 (DIN), D105.1 (DOUT), D105.4 (DIN), D106.1 (DOUT), D106.4 (DIN), D107.1 (DOUT), D107.4 (DIN), D110.1 (DOUT), D110.4 (DIN), D111.1 (DOUT), D111.4 (DIN), D112.1 (DOUT), D112.4 (DIN), D115.1 (DOUT), D115.4 (DIN), D116.1 (DOUT), D116.4 (DIN), D117.1 (DOUT), D117.4 (DIN), D119.1 (DOUT), D119.4 (DIN), D120.1 (DOUT), D120.4 (DIN), D121.1 (DOUT), D121.4 (DIN), D123.1 (DOUT), D123.4 (DIN), D124.1 (DOUT), D124.4 (DIN), D125.1 (DOUT), D125.4 (DIN), D127.1 (DOUT), D127.4 (DIN), D128.1 (DOUT), D128.4 (DIN), D129.1 (DOUT), D129.4 (DIN), D131.1 (DOUT), D131.4 (DIN), D135.1 (DOUT), D135.4 (DIN), D136.4 (DIN), D198.1 (DOUT), D198.4 (DIN), D199.1 (DOUT), D199.4 (DIN), D76.1 (DOUT), D76.4 (DIN), D77.1 (DOUT), D77.4 (DIN), D78.1 (DOUT), D78.4 (DIN), D79.1 (DOUT), D79.4 (DIN), D81.1 (DOUT), D81.4 (DIN), D82.1 (DOUT), D82.4 (DIN), D83.1 (DOUT), D83.4 (DIN), D84.1 (DOUT), D84.4 (DIN), D85.1 (DOUT), D85.4 (DIN), D86.1 (DOUT), D86.4 (DIN), D87.1 (DOUT), D87.4 (DIN), D88.1 (DOUT), D88.4 (DIN), D89.1 (DOUT), D89.4 (DIN), D90.1 (DOUT), D90.4 (DIN), D91.1 (DOUT), D91.4 (DIN), D92.1 (DOUT), D92.4 (DIN), D94.1 (DOUT), D94.4 (DIN), D95.1 (DOUT), D95.4 (DIN), D96.1 (DOUT), D96.4 (DIN), D97.1 (DOUT), D97.4 (DIN)
- new net: D1.1 (DOUT), D1.4 (DIN), D104.1 (DOUT), D104.4 (DIN), D109.1 (DOUT), D109.4 (DIN), D114.1 (DOUT), D114.4 (DIN), D118.1 (DOUT), D118.4 (DIN), D122.1 (DOUT), D122.4 (DIN), D126.1 (DOUT), D126.4 (DIN), D130.1 (DOUT), D130.4 (DIN), D99.1 (DOUT), D99.4 (DIN)

Commit message: idk
Parts:
- removed D1, D100, D101, D102, D103, D104, D105, D106, D107, D108, D109, D110, D111, D112, D113, D114, D115, D116, D117, D118, D119, D120, D121, D122, D123, D124, D125, D126, D127, D128, D129, D130, D131, D132, D133, D134, D135, D136, D198, D199, D39, D50, D66, D67, D76, D77, D78, D79, D80, D81, D82, D83, D84, D85, D86, D87, D88, D89, D90, D91, D92, D93, D94, D95, D96, D97, D98, D99: NeoPixel_THT, LED_SMD:LED_SK6812MINI_PLCC4_3.5x3.5mm_P1.75mm, symbol LED:NeoPixel_THT
Connections:
- net LEDS: no longer names the net of U1.34 (GPIO28_ADC2)
Other:
- note removed: "Led String"
