File: toro-pcb/toro-pcb.kicad_pcb (KiCad board)
At the start: 2 copper layers, 206 parts, among them SW1 Kailh_socket, SW10 Kailh_socket, SW11 Kailh_socket, SW12 Kailh_socket, SW13 Kailh_socket, SW14 Kailh_socket, SW15 Kailh_socket, SW16 Kailh_socket, SW17 Kailh_socket, SW18 Kailh_socket, SW19 Kailh_socket, SW2 RotaryEncoder_Switch, SW20 Kailh_socket, SW21 Kailh_socket, SW22 Kailh_socket, SW23 Kailh_socket, SW24 Kailh_socket, SW25 Kailh_socket, SW26 Kailh_socket, SW27 Kailh_socket, SW28 Kailh_socket, SW29 Kailh_socket, SW3 Kailh_socket, SW30 Kailh_socket, SW31 Kailh_socket, SW32 Kailh_socket, SW33 Kailh_socket, SW34 Kailh_socket, SW35 Kailh_socket, SW36 Kailh_socket, SW37 Kailh_socket, SW38 Kailh_socket, SW4 Kailh_socket, SW40 Kailh_socket, SW41 Kailh_socket, SW42 Kailh_socket, SW43 Kailh_socket, SW44 Kailh_socket, SW45 Kailh_socket, SW46 Kailh_socket, SW47 Kailh_socket, SW48 Kailh_socket, SW49 Kailh_socket, SW5 Kailh_socket, SW51 Kailh_socket, SW52 Kailh_socket, SW53 Kailh_socket, SW54 Kailh_socket, SW55 Kailh_socket, SW56 Kailh_socket, SW57 Kailh_socket, SW58 Kailh_socket, SW59 Kailh_socket, SW6 Kailh_socket, SW60 Kailh_socket, SW61 Kailh_socket, SW62 Kailh_socket, SW63 Kailh_socket, SW64 Kailh_socket, SW65 Kailh_socket, SW67 Kailh_socket, SW68 Kailh_socket, SW69 Kailh_socket, SW7 Kailh_socket, SW71 Kailh_socket, SW72 Kailh_socket, SW73 Kailh_socket, SW8 Kailh_socket, SW9 Kailh_socket, U1 Pico

Commit message: set distance between centers to 19.05mm + add space and footprint for stabilizers
Parts:
- added REF**: Stabilizer_MX_2u, keyswitches.pretty-master:Stabilizer_MX_2u, F.Cu at (304.8, 66.7)
- added REF**: Stabilizer_MX_2u, keyswitches.pretty-master:Stabilizer_MX_2u, F.Cu at (192.4, 142.8)
- added REF**: Stabilizer_MX_2u, keyswitches.pretty-master:Stabilizer_MX_2u, F.Cu at (38.1, 123.8)
- added REF**: Stabilizer_MX_2u, keyswitches.pretty-master:Stabilizer_MX_2u, F.Cu at (110.5, 142.9)
- added REF**: Stabilizer_MX_2u, keyswitches.pretty-master:Stabilizer_MX_2u, F.Cu at (297.2, 104.8)
- moved D135 23.0 mm to (249.7, 147.3)
- moved D70 23.0 mm to (258.2, 145.3)
- moved SW68 23.0 mm to (249.6, 142.9)
- moved D65 21.9 mm to (151.8, 145.1)
- moved D134 21.5 mm to (226.9, 147.2)
- moved D69 21.5 mm to (235.7, 145.3)
- moved SW67 21.5 mm to (226.7, 142.9)
- moved D66 21.3 mm to (142.9, 147.5)
- moved SW64 21.3 mm to (142.9, 142.9)
- moved D67 18.4 mm to (192.6, 147.6)
- moved D68 18.4 mm to (201.3, 145.2)
- moved SW65 18.4 mm to (192.4, 142.8)
- moved D50 15.3 mm to (111.3, 147.2)
- moved D64 15.3 mm to (119.5, 145.1)
- moved SW63 15.3 mm to (110.5, 142.9)
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Connections:
- D80 pad 1: LEDS -> Net-(D100-DIN)
- D80 pad 4: LEDS -> Net-(D100-DIN)

Commit message: big keys
Parts:
- moved REF** 34.3 mm to (144.8, 142.9)
- moved U1 23.7 mm to (62.9, 40.0)
- moved SW68 12.6 mm to (262.3, 142.9)
- moved D70 12.6 mm to (270.8, 145.3)
- moved D135 12.6 mm to (262.3, 147.3)
- moved SW67 11.4 mm to (238.1, 142.9)
- moved D134 11.4 mm to (238.4, 147.2)
- moved D69 11.4 mm to (247.1, 145.3)
- moved D39 9.53 mm to (87.8, 147.2)
- moved D63 9.53 mm to (96.6, 145.0)
- moved SW62 9.52 mm to (87.6, 142.9)
- moved D131 7.62 mm to (303.2, 128.2)
- moved D59 7.62 mm to (311.9, 125.8)
- moved SW59 7.62 mm to (302.9, 123.8)
- moved D67 5.72 mm to (198.3, 147.6)
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Other:
- board outline added: 433.7 x 133.3 mm

Commit message: spacing christ all mighty
Parts:
- moved D72 21.9 mm to (324.6, 144.7)
- moved D104 21.9 mm to (354.6, 90.5)
- moved D118 21.9 mm to (354.3, 109.4)
- moved D30 21.9 mm to (362.8, 88.0)
- moved D45 21.9 mm to (362.8, 106.8)
- moved SW30 21.9 mm to (354.0, 85.7)
- moved SW45 21.9 mm to (354.0, 104.8)
- moved D132 21.8 mm to (334.9, 128.3)
- moved D133 21.8 mm to (354.2, 128.2)
- moved D198 21.8 mm to (335.7, 147.4)
- moved D199 21.8 mm to (354.5, 147.4)
- moved D60 21.8 mm to (343.9, 125.8)
- moved D61 21.8 mm to (362.9, 126.1)
- moved D73 21.8 mm to (343.9, 145.0)
- moved D74 21.8 mm to (363.2, 145.0)
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
Commit message: vertically aligned right side 💀
Parts:
- moved D136 0.20 mm to (316.6, 147.5)
- moved SW69 0.20 mm to (316.2, 142.9)
- moved D72 0.20 mm to (324.8, 144.7)
- moved SW55 0.16 mm to (219.1, 123.8)
- moved D127 0.16 mm to (219.2, 128.3)
- moved D55 0.16 mm to (228.0, 125.8)
- moved D125 0.08 mm to (181.2, 128.3)
- moved D111 0.08 mm to (175.4, 109.5)
- moved D112 0.08 mm to (194.7, 109.6)
- moved D113 0.08 mm to (213.4, 109.6)
- moved D114 0.08 mm to (232.4, 109.3)
- moved D115 0.08 mm to (251.7, 109.1)
- moved D116 0.08 mm to (270.7, 109.1)
- moved D22 0.08 mm to (186.0, 87.9)
- moved D24 0.08 mm to (224.0, 87.9)
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Other:
- board size 433.7 x 133.3 mm -> 369.6 x 133.3 mm

Commit message: move leds to back
Parts:
- D1, D100, D101, D102, D103, D104, D105, D106, D107, D108, D109, D110, D111, D112, D113, D114, D115, D116, D117, D118, D119, D120, D121, D122, D123, D124, D125, D126, D127, D128, D129, D130, D131, D132, D133, D134, D135, D136, D198, D199, D39, D50, D66, D67, D76, D77, D78, D79, D80, D81, D82, D83, D84, D85, D86, D87, D88, D89, D90, D91, D92, D93, D94, D95, D96, D97, D98, D99, U1: moved to B.Cu
- moved U1 11.4 mm to (51.4, 40.0), turned to -90 degrees
- moved D8 8.82 mm to (160.0, 72.6), turned to 87 degrees
- moved SW9 8.77 mm to (176.6, 69.7), turned to 3 degrees
- moved D9 8.52 mm to (185.6, 71.3), turned to 93 degrees
- moved D83 8.51 mm to (177.3, 74.7), turned to -177 degrees
- moved SW10 8.50 mm to (195.6, 68.7), turned to 3 degrees
- moved SW8 8.38 mm to (151.0, 70.0), turned to -3 degrees
- moved SW11 8.34 mm to (214.6, 67.7), turned to 3 degrees
- moved SW12 8.30 mm to (233.6, 66.7), turned to 3 degrees
- moved D10 8.29 mm to (204.6, 70.5), turned to 93 degrees
- moved D84 8.24 mm to (196.2, 73.7), turned to -177 degrees
- moved D11 8.21 mm to (223.5, 69.1), turned to 93 degrees
- moved D82 8.15 mm to (151.0, 74.8), turned to 177 degrees
- moved D136 8.14 mm to (308.5, 147.5), turned to 180 degrees
- moved D85 8.09 mm to (214.9, 72.4), turned to -177 degrees
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Routing:
- net Net-(D5-A): track 0.00 -> 19.6 mm
- net Net-(D6-A): track 0.00 -> 19.5 mm
- net Net-(D13-A): track 0.00 -> 19.5 mm
- net Net-(D15-A): track 0.00 -> 19.4 mm
- net Net-(D8-A): track 0.00 -> 19.2 mm
- net Net-(D2-A): track 0.00 -> 19.1 mm
- net Net-(D3-A): track 0.00 -> 19.0 mm
- net Net-(D14-A): track 0.00 -> 19.0 mm
- net Net-(D7-A): track 0.00 -> 19.0 mm
- net Net-(D4-A): track 0.00 -> 19.0 mm
- net Net-(D12-A): track 0.00 -> 18.9 mm
- net Net-(D10-A): track 0.00 -> 18.8 mm
- net Net-(D9-A): track 0.00 -> 18.8 mm
- net Net-(D11-A): track 0.00 -> 18.6 mm
Other:
- board size 369.6 x 133.3 mm -> 348.6 x 133.4 mm

Commit message: i fucked up
Parts:
- renumbered D62 to D27, D63 to D30, D64 to D31, D65 to D32, D72 to D59, D73 to D60, D74 to D61, D60 to D62, D30 to D63, D45 to D64, D61 to D65, SW61 to SW27, SW62 to SW30, SW63 to SW31, SW64 to SW32, SW69 to SW59, SW71 to SW60, SW72 to SW61, SW73 to SW62, SW30 to SW63, SW45 to SW64, SW60 to SW65
Connections:
- SW27 pad 1: Col 16 -> Col 1
- SW27 pad 2: Net-(D61-A) -> Net-(D27-A)
- SW30 pad 1: Col 15 -> Col 3
- SW30 pad 2: Net-(D62-A) -> Net-(D30-A)
- SW31 pad 1: Col 16 -> Col 4
- SW31 pad 2: Net-(D63-A) -> Net-(D31-A)
- SW32 pad 1: Col 16 -> Col 5
- SW32 pad 2: Net-(D64-A) -> Net-(D32-A)
- SW59 pad 1: Col 11 -> Col 14
- SW59 pad 2: Net-(D70-A) -> Net-(D59-A)
- SW60 pad 1: Col 13 -> Col 15
- SW60 pad 2: Net-(D72-A) -> Net-(D60-A)
- SW61 pad 1: Col 12 -> Col 16
- SW61 pad 2: Net-(D73-A) -> Net-(D61-A)
- SW62 pad 1: Col 12 -> Col 15
- SW62 pad 2: Net-(D74-A) -> Net-(D62-A)
- SW63 pad 1: Col 3 -> Col 16
- SW63 pad 2: Net-(D30-A) -> Net-(D63-A)
- SW64 pad 1: Col 8 -> Col 16
- SW64 pad 2: Net-(D45-A) -> Net-(D64-A)
- SW65 pad 1: Col 15 -> Col 16
- SW65 pad 2: Net-(D60-A) -> Net-(D65-A)
Routing:
- net GND: track 0.00 -> 5.13 mm
- net Net-(D65-A): track 0.00 -> 0.86 mm

Commit message: idk
Parts:
- removed D1, D100, D101, D102, D103, D104, D105, D106, D107, D108, D109, D110, D111, D112, D113, D114, D115, D116, D117, D118, D119, D120, D121, D122, D123, D124, D125, D126, D127, D128, D129, D130, D131, D132, D133, D134, D135, D136, D198, D199, D39, D50, D66, D67, D76, D77, D78, D79, D80, D81, D82, D83, D84, D85, D86, D87, D88, D89, D90, D91, D92, D93, D94, D95, D96, D97, D98, D99: NeoPixel_THT, LED_SMD:LED_SK6812MINI_PLCC4_3.5x3.5mm_P1.75mm
- added G***: LOGO, fun:toro, F.Cu at (157.0, 42.0)
- added G***: LOGO, fun:hackclub, F.Cu at (112.5, 41.5)
- D10: renamed from D17; moved to B.Cu
- D11: renamed from D18; moved to B.Cu
- D12: renamed from D19; moved to B.Cu
- D13: renamed from D20; moved to B.Cu
- D14: renamed from D21; moved to B.Cu
- D15: renamed from D31; moved to B.Cu
- D17: renamed from D33; moved to B.Cu
- D18: renamed from D34; moved to B.Cu
- D19: renamed from D35; moved to B.Cu
- D2, D27, D3, D30, D31, D32 (x2), D4, D5, D59, D6, D60, D61, D62, D63, D64, D65, D7, D8: moved to B.Cu
- D20: renamed from D36; moved to B.Cu
- D21: renamed from D46; moved to B.Cu
- D22: renamed from D47; moved to B.Cu
- D23: renamed from D48; moved to B.Cu
- D24: renamed from D49; moved to B.Cu
- D25: renamed from D51; moved to B.Cu
- D26: renamed from D52; moved to B.Cu
- D28: renamed from D9; moved to B.Cu
- D29: renamed from D10; moved to B.Cu
- D33: renamed from D11; moved to B.Cu
- D34: renamed from D12; moved to B.Cu
- D35: renamed from D13; moved to B.Cu
- D36: renamed from D14; moved to B.Cu
- D37: renamed from D15; moved to B.Cu
- D38: renamed from D22; moved to B.Cu
- D40: renamed from D23; moved to B.Cu
- D41: renamed from D37; moved to B.Cu
- D42: renamed from D24; moved to B.Cu
- D43: renamed from D38; moved to B.Cu
- D44: renamed from D25; moved to B.Cu
- D45: renamed from D40; moved to B.Cu
- D46: renamed from D26; moved to B.Cu
- D47: renamed from D41; moved to B.Cu
- D48: renamed from D27; moved to B.Cu
- D49: renamed from D42; moved to B.Cu
- D51: renamed from D53; moved to B.Cu
- D52: renamed from D54; moved to B.Cu
- D53: renamed from D55; moved to B.Cu
- D54: renamed from D56; moved to B.Cu
- D55: renamed from D57; moved to B.Cu
- D56: renamed from D68; moved to B.Cu
- D57: renamed from D69; moved to B.Cu
- D58: renamed from D70; moved to B.Cu
- D68: renamed from D28; moved to B.Cu
- D69: renamed from D43; moved to B.Cu
- D70: renamed from D58; moved to B.Cu
- D72: renamed from D29; moved to B.Cu
- D73: renamed from D44; moved to B.Cu
- D74: renamed from D59; moved to B.Cu
- D9: renamed from D16; moved to B.Cu
- moved U1 1.91 mm to (53.3, 40.0)
- moved D54 0.91 mm to (241.8, 125.8), turned to 93 degrees
- moved D57 0.55 mm to (243.4, 145.0)
- moved D59 0.15 mm to (317.0, 144.7)
- turned D17 to 90 degrees
- turned D49 to 93 degrees
- renumbered SW17 to SW10, SW18 to SW11, SW19 to SW12, SW20 to SW13, SW31 to SW14, SW21 to SW14, SW32 to SW16, SW33 to SW17, SW34 to SW18, SW35 to SW19, SW36 to SW20, SW46 to SW21, SW47 to SW22, SW48 to SW23, SW49 to SW24, SW51 to SW25, SW52 to SW26, SW9 to SW28, SW10 to SW29, SW11 to SW33, SW12 to SW34, SW13 to SW35, SW14 to SW36, SW15 to SW37, SW22 to SW38, SW23 to SW40, SW37 to SW41, SW24 to SW42, SW38 to SW43, SW25 to SW44, SW40 to SW45, SW26 to SW46, SW27 to SW48, SW42 to SW49, SW53 to SW51, SW54 to SW52, SW55 to SW53, SW56 to SW54, SW57 to SW55, SW65 to SW56, SW67 to SW57, SW41 to SW57, SW68 to SW58, SW28 to SW67, SW43 to SW68, SW58 to SW69, SW29 to SW71, SW44 to SW72, SW59 to SW73, SW16 to SW9
Connections:
- D10 pad 1: Row 2 -> Row 1
- D11 pad 1: Row 2 -> Row 1
- D12 pad 1: Row 2 -> Row 1
- D13 pad 1: Row 2 -> Row 1
- D14 pad 1: Row 3 -> Row 1
- D15 pad 1: Row 4 -> Row 2
- D15 pad 2: Net-(D31-A) -> Net-(D15-A)
- D17 pad 1: Row 0 -> Row 2
- D18 pad 1: Row 0 -> Row 2
- D19 pad 1: Row 0 -> Row 2
- D20 pad 1: Row 0 -> Row 2
- D21 pad 1: Row 1 -> Row 3
- D22 pad 1: Row 2 -> Row 3
- D23 pad 1: Row 1 -> Row 3
- D24 pad 1: Row 2 -> Row 3
- D27 pad 1: Row 3 -> Row 4
- D27 pad 2: Net-(D62-A) -> Net-(D27-A)
- D28 pad 1: Row 1 -> Row 0
- D29 pad 1: Row 1 -> Row 0
- D30 pad 1: Row 1 -> Row 4
- D30 pad 2: Net-(D63-A) -> Net-(D30-A)
- D31 pad 1: Row 2 -> Row 4
- D31 pad 2: Net-(D64-A) -> Net-(D31-A)
- D32 pad 1: Row 4 -> Row 2
- D32 pad 2: Net-(D32-A) -> Net-(D16-A)
- D32 pad 1: Row 3 -> Row 4
- D32 pad 2: Net-(D65-A) -> Net-(D32-A)
- D33 pad 1: Row 1 -> Row 0
- D34 pad 1: Row 1 -> Row 0
- D35 pad 1: Row 1 -> Row 0
- D36 pad 1: Row 1 -> Row 0
- D37 pad 1: Row 2 -> Row 0
- D38 pad 1: Row 3 -> Row 1
- D40 pad 1: Row 3 -> Row 1
- D41 pad 1: Row 0 -> Row 2
- D42 pad 1: Row 3 -> Row 1
- D43 pad 1: Row 1 -> Row 2
- D44 pad 1: Row 3 -> Row 1
- D45 pad 1: Row 1 -> Row 2
- D46 pad 1: Row 3 -> Row 1
- D48 pad 1: Row 4 -> Row 1
- D48 pad 2: Net-(D27-A) -> Net-(D48-A)
- D49 pad 1: Row 1 -> Row 2
- D54 pad 1: Row 4 -> Row 3
- D55 pad 1: Row 4 -> Row 3
- D56 pad 1: Row 1 -> Row 4
- D56 pad 2: Net-(D68-A) (its old number) -> Net-(D56-A)
- D57 pad 1: Row 2 -> Row 4
- D57 pad 2: Net-(D69-A) (its old number) -> Net-(D57-A)
- D58 pad 1: Row 3 -> Row 4
- D58 pad 2: Net-(D70-A) (its old number) -> Net-(D58-A)
- D59 pad 1: Row 1 -> Row 4
- D59 pad 2: Net-(D72-A) (its old number) -> Net-(D59-A)
- D60 pad 1: Row 2 -> Row 4
- D60 pad 2: Net-(D73-A) (its old number) -> Net-(D60-A)
- D61 pad 1: Row 3 -> Row 4
- D61 pad 2: Net-(D74-A) -> Net-(D61-A)
- D62 pad 1: Row 4 -> Row 3
- D62 pad 2: Net-(D60-A) -> Net-(D62-A)
- D63 pad 1: Row 4 -> Row 1
- D63 pad 2: Net-(D30-A) -> Net-(D63-A)
- D64 pad 2: Net-(D45-A) (its old number) -> Net-(D64-A)
- D65 pad 1: Row 4 -> Row 3
- D65 pad 2: Net-(D61-A) -> Net-(D65-A)
- D68 pad 1: Row 0 -> Row 1
- D70 pad 1: Row 4 -> Row 3
- D72 pad 1: Row 0 -> Row 1
- D73 pad 1: Row 1 -> Row 2
- D74 pad 1: Row 4 -> Row 3
- D74 pad 2: Net-(D59-A) -> Net-(D74-A)
- D9 pad 1: Row 2 -> Row 1
- SW10 pad 1: Col 2 -> Col 1
- SW11 pad 1: Col 3 -> Col 2
- SW12 pad 1: Col 4 -> Col 3
- SW13 pad 1: Col 5 -> Col 4
- SW14 pad 1: Col 4 -> Col 0
- SW14 pad 2: Net-(D31-A) -> Net-(D15-A)
- SW14 pad 1: Col 0 -> Col 5
- SW16 pad 1: Col 5 -> Col 1
- SW16 pad 2: Net-(D32-A) -> Net-(D16-A)
- SW17 pad 1: Col 9 -> Col 2
- SW18 pad 1: Col 10 -> Col 3
- SW19 pad 1: Col 11 -> Col 4
- SW20 pad 1: Col 12 -> Col 5
- SW21 pad 1: Col 10 -> Col 0
- SW22 pad 1: Col 9 -> Col 1
- SW23 pad 1: Col 11 -> Col 2
- SW24 pad 1: Col 10 -> Col 3
- SW25 pad 1: Col 6 -> Col 4
- SW26 pad 1: Col 7 -> Col 5
- SW27 pad 1: Col 1 -> Col 0
- SW28 pad 1: Col 0 -> Col 7
- SW29 pad 1: Col 1 -> Col 8
- SW33 pad 1: Col 2 -> Col 9
- SW34 pad 1: Col 3 -> Col 10
- SW35 pad 1: Col 4 -> Col 11
- SW36 pad 1: Col 5 -> Col 12
- SW37 pad 1: Col 0 -> Col 13
- SW38 pad 1: Col 1 -> Col 6
- SW40 pad 1: Col 2 -> Col 7
- SW41 pad 1: Col 13 -> Col 6
- SW42 pad 1: Col 3 -> Col 8
- SW43 pad 1: Col 6 -> Col 7
- SW44 pad 1: Col 4 -> Col 9
- SW45 pad 1: Col 7 -> Col 8
- SW46 pad 1: Col 5 -> Col 10
- SW48 pad 1: Col 0 -> Col 11
- SW48 pad 2: Net-(D27-A) -> Net-(D48-A)
- SW49 pad 1: Col 8 -> Col 10
- SW51 pad 1: Col 8 -> Col 6
- SW52 pad 1: Col 9 -> Col 7
- SW53 pad 1: Col 10 -> Col 8
- SW54 pad 1: Col 6 -> Col 9
- SW55 pad 1: Col 7 -> Col 10
- SW56 pad 1: Col 16 -> Col 6
- SW56 pad 2: Net-(D65-A) -> Net-(D56-A)
- SW57 pad 1: Col 12 -> Col 7
- SW57 pad 2: Net-(D68-A) (its old number) -> Net-(D57-A)
- SW57 pad 1: Col 6 -> Col 9
- SW58 pad 1: Col 11 -> Col 8
- SW58 pad 2: Net-(D69-A) (its old number) -> Net-(D58-A)
- SW67 pad 1: Col 7 -> Col 12
- SW68 pad 1: Col 7 -> Col 11
- SW69 pad 1: Col 8 -> Col 11
- SW71 pad 1: Col 8 -> Col 13
- SW72 pad 1: Col 9 -> Col 12
- SW73 pad 1: Col 14 -> Col 12
- SW73 pad 2: Net-(D59-A) -> Net-(D74-A)
- SW9 pad 1: Col 1 -> Col 0
Routing:
- net Row 4: track 0.00 -> 474.8 mm
- net Row 3: track 0.00 -> 448.9 mm
- net Row 2: track 0.00 -> 427.4 mm
- net Row 1: track 0.00 -> 402.8 mm
- net Col 16: track 0.00 -> 370.9 mm, vias 0 -> 5
- net Col 15: track 0.00 -> 340.2 mm, vias 0 -> 3
- net Col 14: track 0.00 -> 331.9 mm, vias 0 -> 2
- net Row 0: track 0.00 -> 328.7 mm
- net ENC_S1: track 0.00 -> 316.4 mm, vias 0 -> 1
- net ENC_B: track 0.00 -> 307.4 mm, vias 0 -> 1
- net ENC_A: track 0.00 -> 295.5 mm, vias 0 -> 2
- net Col 12: track 0.00 -> 286.5 mm, vias 0 -> 7
- net Col 13: track 0.00 -> 269.2 mm, vias 0 -> 3
- net Col 8: track 0.00 -> 261.8 mm, vias 0 -> 6
- net Col 11: track 0.00 -> 259.9 mm, vias 0 -> 7
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Other:
- board size 348.6 x 133.4 mm -> 341 x 138.2 mm
- board text added: "toro-board v.1!!"

Commit message: cad
Parts:
- moved SW2 2.62 mm to (341.8, 58.2)
Routing:
- net ENC_B: track 307.4 -> 304.7 mm, vias 1 -> 2
- net ENC_A: track 295.5 -> 292.8 mm
- net ENC_S1: track 316.4 -> 315.3 mm
- net Col 10: track 245.4 -> 244.8 mm, vias 5 -> 7
