File: toro-pcb/toro-pcb.kicad_pcb (KiCad board)
At the start: 2 copper layers, 341 x 138.2 mm, 145 parts, among them SW1 Kailh_socket, SW10 Kailh_socket, SW11 Kailh_socket, SW12 Kailh_socket, SW13 Kailh_socket, SW14 Kailh_socket, SW16 Kailh_socket, SW17 Kailh_socket, SW18 Kailh_socket, SW19 Kailh_socket, SW2 RotaryEncoder_Switch, SW20 Kailh_socket, SW21 Kailh_socket, SW22 Kailh_socket, SW23 Kailh_socket, SW24 Kailh_socket, SW25 Kailh_socket, SW26 Kailh_socket, SW27 Kailh_socket, SW28 Kailh_socket, SW29 Kailh_socket, SW3 Kailh_socket, SW30 Kailh_socket, SW31 Kailh_socket, SW32 Kailh_socket, SW33 Kailh_socket, SW34 Kailh_socket, SW35 Kailh_socket, SW36 Kailh_socket, SW37 Kailh_socket, SW38 Kailh_socket, SW4 Kailh_socket, SW40 Kailh_socket, SW41 Kailh_socket, SW42 Kailh_socket, SW43 Kailh_socket, SW44 Kailh_socket, SW45 Kailh_socket, SW46 Kailh_socket, SW48 Kailh_socket, SW49 Kailh_socket, SW5 Kailh_socket, SW51 Kailh_socket, SW52 Kailh_socket, SW53 Kailh_socket, SW54 Kailh_socket, SW55 Kailh_socket, SW56 Kailh_socket, SW57 Kailh_socket, SW58 Kailh_socket, SW59 Kailh_socket, SW6 Kailh_socket, SW60 Kailh_socket, SW61 Kailh_socket, SW62 Kailh_socket, SW63 Kailh_socket, SW64 Kailh_socket, SW65 Kailh_socket, SW67 Kailh_socket, SW68 Kailh_socket, SW69 Kailh_socket, SW7 Kailh_socket, SW71 Kailh_socket, SW72 Kailh_socket, SW73 Kailh_socket, SW8 Kailh_socket, SW9 Kailh_socket, U1 Pico

Commit message: iiiiiuhhhuhhh rewiring
Parts:
- moved G*** 9.06 mm to (148.0, 43.0)
- moved D8 8.47 mm to (158.3, 80.9), turned to 82 degrees
- moved D26 7.65 mm to (156.3, 137.4), turned to 82 degrees
- moved SW26 6.99 mm to (148.1, 134.1), turned to -8 degrees
- moved D32 6.97 mm to (148.3, 155.4), turned to 82 degrees
- moved D20 6.54 mm to (149.3, 116.7), turned to 82 degrees
- moved U1 6.40 mm to (50.5, 45.7)
- moved REF** 6.19 mm to (139.8, 152.2), turned to 172 degrees
- moved SW32 6.18 mm to (139.7, 152.1), turned to -8 degrees
- moved SW51 6.11 mm to (174.2, 132.9), turned to 8 degrees
- moved D25 6.08 mm to (137.5, 134.8), turned to 82 degrees
- moved SW8 5.97 mm to (149.8, 75.9), turned to -8 degrees
- moved D14 5.86 mm to (145.1, 97.2), turned to 82 degrees
- moved SW20 5.85 mm to (140.8, 113.5), turned to -8 degrees
- moved SW38 5.74 mm to (169.9, 94.9), turned to 8 degrees
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Routing:
- net Col 15: track 340.2 -> 354.5 mm, vias 3 -> 4
- net Col 14: track 331.9 -> 339.4 mm
- net Col 8: track 261.8 -> 268.6 mm, vias 6 -> 5
- net Col 0: track 114.2 -> 107.5 mm, vias 6 -> 5
- net Col 5: track 176.0 -> 181.7 mm, vias 6 -> 5
- net ENC_B: track 304.7 -> 299.1 mm, vias 2 -> 1
- net Col 10: track 244.8 -> 250.0 mm, vias 7 -> 4
- net Row 0: track 328.7 -> 332.6 mm
- net Col 3: track 162.3 -> 159.0 mm
- net Col 16: track 370.9 -> 373.9 mm
- net Net-(D35-A): track 19.1 -> 22.1 mm
- net Col 1: track 99.7 -> 102.6 mm, vias 5 -> 4
- net Col 4: track 175.3 -> 172.5 mm, vias 6 -> 5
- net Net-(D6-A): track 19.0 -> 21.7 mm
- net Row 4: track 474.8 -> 472.6 mm
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Other:
- board size 341 x 138.2 mm -> 339.2 x 137 mm
